File: quiz_remote_compact/quiz_remote.kicad_pcb (KiCad board)
At the start: 2 copper layers, 52 x 90 mm, 127 parts, among them J1 LUA_SOCKET_ROW_A, J2 LUA_SOCKET_ROW_B, SW1 6x6_THT_NO, SW10 6x6_THT_NO, SW11 6x6_THT_NO, SW12 6x6_THT_NO, SW13 6x6_THT_NO, SW14 6x6_THT_NO, SW15 6x6_THT_NO, SW16 6x6_THT_NO, SW2 6x6_THT_NO, SW3 6x6_THT_NO, SW4 6x6_THT_NO, SW5 6x6_THT_NO, SW6 6x6_THT_NO, SW7 6x6_THT_NO, SW8 6x6_THT_NO, SW9 6x6_THT_NO, U1 MT3608L, U2 74HC595D,118

Commit message: Add M2 mounting holes with copper keep-out, add single-sided board and Gerber outputs
Parts:
- added H1: MountingHole_2.2mm_M2, MountingHole_2.2mm_M2, F.Cu at (102.0, 69.8)
- added H2: MountingHole_2.2mm_M2, MountingHole_2.2mm_M2, F.Cu at (149.2, 70.5)
- added H3: MountingHole_2.2mm_M2, MountingHole_2.2mm_M2, F.Cu at (103.5, 138.1)
- added H4: MountingHole_2.2mm_M2, MountingHole_2.2mm_M2, F.Cu at (149.8, 138.1)
